File: hardware/rev_a/MCU_Board.kicad_sch (KiCad schematic)
At the start: 28 parts, among them J1 ST-Link, J2 Conn_01x08, J3 Bus, J4 Conn_01x08, J5 Conn_02x07_Odd_Even, SW1 nRST, U1 STM32F042K6Tx, U3 SN65HVD230, U4 LP2985-3.3, Y1 8Mhz

Commit message: Fix all the warnings or errors and add the 'fab' folder with all the required files for production.
Parts:
- D4: footprint digikey-footprints:DO-214AC -> custom:DO-214AA
- J1: footprint Connector_PinHeader_2.54mm:PinHeader_1x04_P2.54mm_Vertical -> custom:st-link
- J2, J4: footprint Connector_PinHeader_2.54mm:PinHeader_1x08_P2.54mm_Vertical -> custom:CONN_01x08
- J3: footprint Connector_Phoenix_MSTB:PhoenixContact_MSTBVA_2,5_4-G-5,08_1x04_P5.08mm_Vertical -> custom:PhoenixContact_MSTBVA_2,5_4-G-5,08_1x04_P5.08mm_Vertical_custom
- J5: footprint Connector_PinHeader_2.54mm:PinHeader_2x07_P2.54mm_Vertical -> custom:addr_jumpers
Changed lines of the file:
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@@
       (effects (font (size 1.27 1.27)) (justify left) hide)
     )
-    (property "Footprint" "Connector_PinHeader_2.54mm:PinHeader_1x04_P2.54mm_Vertical" (at 158.75 45.72 0)
+    (property "Footprint" "custom:st-link" (at 158.75 45.72 0)
       (effects (font (size 1.27 1.27)) hide)
     )
@@
       (effects (font (size 1.27 1.27)) (justify left))
     )
-    (property "Footprint" "Connector_Phoenix_MSTB:PhoenixContact_MSTBVA_2,5_4-G-5,08_1x04_P5.08mm_Vertical" (at 273.05 39.37 0)
+    (property "Footprint" "custom:PhoenixContact_MSTBVA_2,5_4-G-5,08_1x04_P5.08mm_Vertical_custom" (at 273.05 39.37 0)
       (effects (font (size 1.27 1.27)) hide)
     )
@@
       (effects (font (size 1.27 1.27)) (justify left) hide)
     )
-    (property "Footprint" "Connector_PinHeader_2.54mm:PinHeader_1x08_P2.54mm_Vertical" (at 231.14 85.09 0)
+    (property "Footprint" "custom:CONN_01x08" (at 231.14 85.09 0)
       (effects (font (size 1.27 1.27)) hide)
     )
@@
       (effects (font (size 1.27 1.27)) (justify left) hide)
     )
-    (property "Footprint" "Connector_PinHeader_2.54mm:PinHeader_1x08_P2.54mm_Vertical" (at 236.22 85.09 0)
+    (property "Footprint" "custom:CONN_01x08" (at 236.22 85.09 0)
       (effects (font (size 1.27 1.27)) hide)
     )
@@
       (effects (font (size 1.27 1.27)) hide)
     )
-    (property "Footprint" "Connector_PinHeader_2.54mm:PinHeader_2x07_P2.54mm_Vertical" (at 133.35 74.93 0)
+    (property "Footprint" "custom:addr_jumpers" (at 133.35 74.93 0)
       (effects (font (size 1.27 1.27)) hide)
     )
@@
       (effects (font (size 1.524 1.524)) (justify right))
     )
-    (property "Footprint" "digikey-footprints:DO-214AC" (at 254 45.72 0)
+    (property "Footprint" "custom:DO-214AA" (at 254 45.72 0)
       (effects (font (size 1.524 1.524)) (justify left) hide)
     )
