File: hardware/rev_a/MCU_Board.kicad_pcb (KiCad board)
At the start: 2 copper layers, 50.8 x 55.9 mm, 35 parts, among them J1 ST-Link, J2 Conn_01x08, J3 Bus, J4 Conn_01x08, J5 Conn_02x07_Odd_Even, SW1 nRST, U2 MC34063AD, U3 SN65HVD230, U5 STM32F042K6Tx, Y1 8Mhz

Commit message: Version under review by PCBWay (Nucleo Shield)
Parts:
- removed C2: 18p, Capacitor_SMD:C_0805_2012Metric_Pad1.18x1.45mm_HandSolder
- removed C3, C7, C8, C9: 100n, Capacitor_SMD:C_0805_2012Metric_Pad1.18x1.45mm_HandSolder
- removed FB1: FerriteBead, Inductor_SMD:L_0805_2012Metric_Pad1.05x1.20mm_HandSolder
- removed J4: Conn_01x08, custom:CONN_01x08
- removed R1: 100k, Resistor_SMD:R_0805_2012Metric_Pad1.20x1.40mm_HandSolder
- removed SW1: nRST, Button_Switch_SMD:SW_SPST_B3U-1000P-B
- removed U5: STM32F042K6Tx, Package_QFP:LQFP-32_7x7mm_P0.8mm
- removed Y1: 8Mhz, Crystal:Crystal_HC18-U_Vertical
- added J6: Conn_01x15, Connector_PinHeader_2.54mm:PinHeader_1x15_P2.54mm_Vertical, F.Cu at (54.6, 158.8)
- added J7: Conn_01x15, Connector_PinHeader_2.54mm:PinHeader_1x15_P2.54mm_Vertical, F.Cu at (54.6, 137.2)
- C1: value 18p -> 100n; footprint Capacitor_SMD:C_0805_2012Metric_Pad1.18x1.45mm_HandSolder -> Capacitor_THT:C_Disc_D5.0mm_W2.5mm_P5.00mm
- C10: footprint Capacitor_SMD:C_0805_2012Metric_Pad1.18x1.45mm_HandSolder -> Capacitor_THT:C_Disc_D5.0mm_W2.5mm_P5.00mm
- C4: value 470p -> 680p; footprint Capacitor_SMD:C_0805_2012Metric_Pad1.18x1.45mm_HandSolder -> Capacitor_THT:C_Disc_D5.0mm_W2.5mm_P5.00mm
- J1: value ST-Link -> Conn_01x15; footprint custom:st-link -> Connector_PinHeader_2.54mm:PinHeader_1x15_P2.54mm_Vertical
- J2: value Conn_01x08 -> Conn_01x02; footprint custom:CONN_01x08 -> Connector_PinHeader_2.54mm:PinHeader_1x02_P2.54mm_Vertical
- J5: value Conn_02x07_Odd_Even -> Conn_01x15; footprint custom:addr_jumpers -> Connector_PinHeader_2.54mm:PinHeader_1x15_P2.54mm_Vertical
- R2, R4: footprint Resistor_SMD:R_0805_2012Metric_Pad1.20x1.40mm_HandSolder -> Resistor_THT:R_Axial_DIN0309_L9.0mm_D3.2mm_P2.54mm_Vertical
- R3: value 0R47 -> 0R33; footprint Resistor_SMD:R_0805_2012Metric_Pad1.20x1.40mm_HandSolder -> Resistor_THT:R_Axial_DIN0309_L9.0mm_D3.2mm_P2.54mm_Vertical
- R5: value 10k -> 6k2; footprint Resistor_SMD:R_0805_2012Metric_Pad1.20x1.40mm_HandSolder -> Resistor_THT:R_Axial_DIN0309_L9.0mm_D3.2mm_P2.54mm_Vertical
- R6: value 6k2 -> 10k; footprint Resistor_SMD:R_0805_2012Metric_Pad1.20x1.40mm_HandSolder -> Resistor_THT:R_Axial_DIN0309_L9.0mm_D3.2mm_P2.54mm_Vertical
- moved J5 38.2 mm to (90.2, 165.1), turned to -90 degrees
- moved C6 28.2 mm to (81.1, 128.3), turned to 180 degrees
- moved L1 26.0 mm to (80.9, 114.3), turned to -90 degrees
- moved J1 22.9 mm to (90.2, 143.5)
- moved C1 21.3 mm to (83.9, 133.3), turned to 0 degrees
- moved C10 13.9 mm to (88.9, 127.6), turned to 0 degrees
- moved R2 9.84 mm to (87.5, 122.2), turned to 90 degrees
- moved D2 9.70 mm to (93.3, 112.4), turned to -90 degrees
- moved U3 6.37 mm to (92.7, 121.3), turned to 90 degrees
- moved R5 5.19 mm to (56.8, 130.8)
- moved R6 5.13 mm to (66.0, 130.8)
- moved C4 4.88 mm to (74.3, 114.3), turned to -90 degrees
- moved R3 4.10 mm to (66.0, 125.7)
- moved J2 2.84 mm to (49.5, 129.5), turned to 180 degrees
- moved JP1 2.58 mm to (91.4, 101.6), turned to 90 degrees
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Connections:
- C1 pad 1: Net-(U5-PF0) -> GND
- C1 pad 2: GND -> /NUCLEO_+3V3
- C10 pad 2: /VDD -> /NUCLEO_+3V3
- C6 pad 1: /VDD -> /NUCLEO_+3V3
- J1 pad 1: GND -> /NUCLEO_PB3
- J1 pad 2: /VDD -> /NUCLEO_+3V3
- J1 pad 3: /SWDIO -> /NUCLEO_AREF
- J1 pad 4: /SWCLK -> /NUCLEO_PA0
- J2 pad 1: /VDD -> GND
- J2 pad 2: /PA15 -> Net-(D5-K)
- J5 pad 1: /ADDR_1 -> /NUCLEO_PB4
- J5 pad 10: GND -> /NUCLEO_PB0
- J5 pad 11: /ADDR_32 -> /NUCLEO_PA12
- J5 pad 13: /ADDR_64 -> /NUCLEO_NRST
- J5 pad 14: GND -> /NUCLEO_PA10
- J5 pad 2: GND -> /NUCLEO_PB5
- J5 pad 3: /ADDR_2 -> /NUCLEO_PA11
- J5 pad 4: GND -> /NUCLEO_PA8
- J5 pad 5: /ADDR_4 -> /NUCLEO_PC15
- J5 pad 6: GND -> /NUCLEO_PC14
- J5 pad 7: /ADDR_8 -> /NUCLEO_PB1
- J5 pad 8: GND -> /NUCLEO_PB6
- J5 pad 9: /ADDR_16 -> /NUCLEO_PB7
- L1 pad 2: /VDD -> /NUCLEO_+3V3
- R6 pad 2: /VDD -> /NUCLEO_+3V3
- U3 pad 1: /CAN_TX -> /NUCLEO_PA12
- U3 pad 3: /VDD -> /NUCLEO_+3V3
- U3 pad 4: /CAN_RX -> /NUCLEO_PA11
Routing:
- net /VDD: track 176.6 -> 0.00 mm
- net GND: track 285.5 -> 216.1 mm
- net /NUCLEO_PA12: track 0.00 -> 69.0 mm
- net /NUCLEO_+3V3: track 0.00 -> 66.1 mm
- net /nRST: track 63.4 -> 0.00 mm
- net /VIN: track 78.9 -> 24.8 mm
- net /NUCLEO_PA11: track 0.00 -> 50.1 mm
- net /PB7: track 28.2 -> 0.00 mm
- net /NUCLEO_NRST: track 0.00 -> 27.9 mm
- net /PA15: track 27.7 -> 0.00 mm
- net /PB6: track 27.1 -> 0.00 mm
- net /PB3: track 26.9 -> 0.00 mm
- net /PB5: track 26.4 -> 0.00 mm
- net /PB4: track 26.0 -> 0.00 mm
- net /CAN_TX: track 24.8 -> 0.00 mm
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Other:
- board size 50.8 x 55.9 mm -> 50.8 x 68.6 mm
- board text added: "3V3"
- board text added: "5V"
- board text added: "AREF"
- board text added: "NRST"
- board text added: "PA0"
- board text added: "PA1"
- board text added: "PA10"
- board text added: "PA11"
- board text added: "PA12"
- board text added: "PA2"
- board text added: "PA3"
- board text added: "PA4"
- board text added: "PA5"
- board text added: "PA6"
- board text added: "PA7"
- board text added: "PA8"
- board text added: "PA9"
- board text added: "PB0"
- board text added: "PB1"
- board text added: "PB3"
- board text added: "PB4"
- board text added: "PB5"
- board text added: "PB6"
- board text added: "PB7"
- board text added: "PC14"
- board text added: "PC15"
- board text added: "VIN"
- board text added: "Vin(fuse)"
- board text removed: "1"
- board text removed: "64"
- board text removed: "STM32-CAN-Bus-board Rev: A"
- board text removed: "gnd"
- board text removed: "swclk"
- board text removed: "swdio"
- board text removed: "vdd"
